Commit message: Revert "body 를 base_footprint 와 같은 중심좌표(x, y)에 오도록 top_y 확정"
This reverts commit 5e670b293d8cfaddb5180110efcca688c562d5c6.

File: src/description/urdf/vehicle.urdf.xacro (robot description, xacro)
@@ -33,14 +33,12 @@
   <xacro:property name="rear_rpy"  value="0 0 ${-pi/2}"/>
   <!-- top: 예전 static TF 에는 이 라이다가 없다.
-       x, y 는 제약으로 확정: body(=top 내부 IMU)가 base_footprint 와 중심좌표
-       (x, y)가 같아야 한다. top 이 누워 있어 내부 IMU 오프셋도 같이 돈다.
-         R_mount * (0.011, 0.02329, -0.04412) = (-0.011, 0.04412, -0.02329)
-         body_xy = top_xy + (-0.011, 0.04412) = (0, 0)
-         -> top_xy = (0.011, -0.04412)
-       z 만 추정치다(0.8465, 오차 +-0.025). z 는 마스트 높이라 x/y 처럼 0 으로
-       둘 수 없다 - 0 으로 두면 IMU 가 차량 중심에 있다고 모델링되어 회전 시
-       lever arm 이 사라지고 FAST-LIO 의 자세 추정이 틀어진다.
+       x 는 제약으로 확정: body(=내부 IMU)가 base_footprint 와 x 가 같아야 한다.
+       R_mount * (0.011, 0.02329, -0.04412) = (-0.011, 0.04412, -0.02329) 이므로
+       body_x = top_x - 0.011 = 0  ->  top_x = 0.011.
+       y, z 는 아직 추정치다. rbio 값 (0, -0.56, 1.40) 을 front/rear 두 기준의
+       평균 오프셋만큼 되돌린 값이고, front/rear 각각으로 구한 오프셋이 y 에서
+       13cm 어긋나 불확실도가 +-(0.065, 0.025) 다.
        회전은 실측 확인됨(roll -90, yaw 180). -->
-  <xacro:property name="top_xyz"   value="0.011 -0.04412 0.8465"/>
+  <xacro:property name="top_xyz"   value="0.011 -0.275 0.8465"/>
   <xacro:property name="top_rpy"   value="${-pi/2} 0 ${pi}"/>
   <!-- body(=top 라이다 내부 IMU) 에서 본 base_footprint.
@@ -49,5 +47,5 @@
        top_xyz 를 고치면 이 값과 fast_lio*/config/mid360.yaml 의 extrinsic_T 를
        같이 다시 계산해야 한다. -->
-  <xacro:property name="bf_from_body_xyz" value="0.0 0.82321 0.0"/>
+  <xacro:property name="bf_from_body_xyz" value="0.0 0.82321 -0.23088"/>
   <xacro:property name="bf_from_body_rpy" value="${-pi/2} 0 ${-pi}"/>
   <material name="grey"><color rgba="0.4 0.4 0.4 0.5"/></material>
