Commit message: livox_top 장착값을 rbio 캘리브레이션에서 가져오고, 겹쳐보기용 rviz 설정 추가
rbio/TransferRobot-Hanyang-main 의 LidarMountCalibration.cpp 에 라이다 3대
장착값이 전부 들어 있었다. lidarIndex 1 = /livox/lidar_192_168_1_135 = top.

  case 1: {0.0f, -0.56f, 1.40f, -90.0f, 0.0f, 180.0f}   <- top
  case 2: {0.30f,  0.0f, 0.397f,  0.0f, 0.0f,  90.0f}   <- front(navigation)
  case 3: {-0.98f,-0.56f, 0.35f,  0.0f, 0.0f, -90.0f}   <- rear

회전 합성이 yaw*pitch*roll 이라 URDF rpy 와 같은 관례고, roll -90 / yaw 180 은
알려주신 값과 정확히 일치한다. top_xyz 에 (0.0, -0.56, 1.40) 을 넣었다.

다만 같은 파일의 front/rear 병진이 우리 static TF 와 다르다. yaw 는 90/-90 로
일치하는데 xyz 만 어긋나므로 원점 관례 차이로 보인다(rbio 주석이 lidar 2 를
"body -> base_footprint TF 에서 복원" 이라고 한다). top_xyz 도 같은 기준일 수
있어 xacro 에 주석으로 남겼다.

description/rviz/frames_check.rviz 추가: RobotModel + TF + 병합 클라우드를 한
화면에 띄워 URDF 형상과 실제 클라우드가 맞는지 눈으로 확인하는 용도.

Co-Authored-By: Claude Opus 5 (1M context) <noreply@anthropic.com>

File: src/description/urdf/vehicle.urdf.xacro (robot description, xacro)
@@ -25,8 +25,12 @@
   <xacro:property name="rear_xyz"  value="-0.6 -0.34 -0.18"/>
   <xacro:property name="rear_rpy"  value="0 0 ${-pi/2}"/>
-  <!-- top: roll -90도, yaw 180도로 눕혀서 장착.
-       TODO 위치(xyz)가 아직 실측 전이다. 0 0 0 은 임시값이므로
-       FAST-LIO 의 extrinsic 을 확정하기 전에 반드시 채워야 한다. -->
-  <xacro:property name="top_xyz"   value="0 0 0"/>
+  <!-- top: 옆으로 눕혀 장착(roll -90, yaw 180). 원시 -Y 가 중력 방향이 된다.
+       값 출처: rbio TransferRobot LidarMountCalibration.cpp 의 lidarIndex 1
+         return {0.0f, -0.56f, 1.40f, -90.0f, 0.0f, 180.0f};
+       회전 합성이 yaw*pitch*roll (= Rz*Ry*Rx) 라 URDF rpy 와 같은 관례다.
+       주의: 같은 파일의 front/rear 값은 아래 우리 값과 병진이 다르다
+       (rbio 는 base_footprint 기준으로 보인다). 아래 top_xyz 도 그 기준일 수
+       있으므로 RViz 겹쳐보기로 확인이 필요하다. -->
+  <xacro:property name="top_xyz"   value="0.0 -0.56 1.40"/>
   <xacro:property name="top_rpy"   value="${-pi/2} 0 ${pi}"/>
   <!-- MID-360 몸통 원점에서 내부 IMU 까지 (Livox 공장값) -->

Commit message: 장착값을 rbio 기준으로 통일하고, body 가 IMU 프레임이라는 점을 반영
[body 는 차량 기준점이 아니다]
FAST-LIO 의 "body" 는 IMU 프레임이다. publish_frame_body 가
RGBpointBodyLidarToIMU 로 포인트를 IMU 좌표로 옮긴 뒤 body 로 stamp 한다.
IMU 가 상단 라이다 안에 있으므로 body 는 마스트 위 1.4m, 측방 0.56m 지점이다.

이걸 모르고 짜여 있던 것들:
- URDF 를 body 루트에 차량 형상으로 그려놨었다 -> body 아래 base_footprint 를
  두고 센서를 거기 매다는 구조로 변경. TF 는 프레임당 부모가 하나뿐이라
  FAST-LIO 가 소유한 body 가 루트일 수밖에 없다.
- tf_2d.py 가 body 를 평면화하고 있었다 -> base_footprint 로 변경. 그대로
  두면 base_link 가 마스트 위에 생겨서 nav2 footprint 가 0.56m 어긋난다.

[rbio 기준 통일]
livox_merge 의 extrinsic 을 rbio LidarMountCalibration.cpp 값으로 교체했다.
기존 lidar_1 값은 축 (0.615, 0, 0.789) 기준 180도 회전으로, rbio 나 static TF
어느 쪽과도 맞지 않던 값이다.

  lidar_0 front  base_footprint <- (0.30, 0, 0.397) yaw 90
  lidar_1 rear   base_footprint <- (-0.98, -0.56, 0.35) yaw -90

output.frame_id 를 body -> base_footprint 로. 위 extrinsic 이 실제로 보내는
프레임이 그쪽인데 라벨만 body 였다.

FAST-LIO extrinsic 도 다시 계산했다. 입력이 base_footprint 로 병합된 클라우드이고
IMU 는 livox_top 안에 있으므로, 한 대짜리 공장 오프셋이 아니라 전체 변환이다.
  extrinsic_T: [-0.011, 1.37671, -0.51588]
  extrinsic_R: base_footprint -> IMU 회전

Co-Authored-By: Claude Opus 5 (1M context) <noreply@anthropic.com>

File: src/description/urdf/vehicle.urdf.xacro (robot description, xacro)
@@ -1,15 +1,19 @@
 <?xml version="1.0"?>
 <!--
-  차량 + 센서 장착 형상.
-  여기가 TF 의 유일한 출처다. 예전에는 msg_Multi_launch.py 안에
-  static_transform_publisher 를 늘어놓았는데, 값이 여러 군데로 흩어지고
-  노드 이름이 겹치는 문제가 있었다.
-  프레임 트리:
-    body ─┬─ livox_frame ─┬─ livox_top ── imu_link
-          │               ├─ livox_front
-          │               └─ livox_rear
-          └─ (base_link 은 여기 없음. tf_2d.py 가 odom 밑에 만든다)
-  body 와 livox_frame 은 같은 지점이다. 드라이버가 포인트클라우드 header 에
-  livox_frame 을 찍기 때문에 이름을 남겨둔다.
+  차량 + 센서 장착 형상. TF 의 유일한 출처.
+  장착값 출처: rbio TransferRobot LidarMountCalibration.cpp defaultMountTransform()
+  회전 합성이 yaw*pitch*roll (= Rz*Ry*Rx) 라 URDF rpy 와 같은 관례다.
+  트리가 base_footprint 가 아니라 body 에서 시작하는 이유:
+    FAST-LIO 의 "body" 는 차량 기준점이 아니라 IMU 프레임이다.
+    (publish_frame_body 가 RGBpointBodyLidarToIMU 로 변환해서 body 로 stamp)
+    FAST-LIO 가 camera_init->body 를 이미 내보내므로 body 가 이 URDF 의 루트가
+    되어야 하고, 차량 기준점은 그 아래에 매달린다. TF 는 프레임당 부모가
+    하나뿐이라 반대로는 못 짠다.
+    map ─┬─ camera_init ── body(=IMU, livox_top 내부)
+         │                  └─ base_footprint ─┬─ livox_frame
+         │                                     ├─ livox_top
+         │                                     ├─ livox_front
+         │                                     └─ livox_rear
+         └─ odom ── base_link      <- tf_2d.py 가 base_footprint 를 평면화한 것
 -->
 <robot xmlns:xacro="http://www.ros.org/wiki/xacro" name="vehicle">
@@ -18,25 +22,18 @@
   <xacro:property name="body_width"  value="0.952"/>
   <xacro:property name="body_height" value="0.60"/>
-  <!-- ===== 라이다 장착 ===== -->
-  <!-- front: livox_frame 기준 yaw +90도 -->
-  <xacro:property name="front_xyz" value="0.697 0.35 -0.18"/>
-  <xacro:property name="front_rpy" value="0 0 ${pi/2}"/>
-  <!-- rear: livox_frame 기준 yaw -90도 -->
-  <xacro:property name="rear_xyz"  value="-0.6 -0.34 -0.18"/>
-  <xacro:property name="rear_rpy"  value="0 0 ${-pi/2}"/>
-  <!-- top: 옆으로 눕혀 장착(roll -90, yaw 180). 원시 -Y 가 중력 방향이 된다.
-       값 출처: rbio TransferRobot LidarMountCalibration.cpp 의 lidarIndex 1
-         return {0.0f, -0.56f, 1.40f, -90.0f, 0.0f, 180.0f};
-       회전 합성이 yaw*pitch*roll (= Rz*Ry*Rx) 라 URDF rpy 와 같은 관례다.
-       주의: 같은 파일의 front/rear 값은 아래 우리 값과 병진이 다르다
-       (rbio 는 base_footprint 기준으로 보인다). 아래 top_xyz 도 그 기준일 수
-       있으므로 RViz 겹쳐보기로 확인이 필요하다. -->
+  <!-- ===== 라이다 장착 (base_footprint 기준, rbio 값) ===== -->
   <xacro:property name="top_xyz"   value="0.0 -0.56 1.40"/>
   <xacro:property name="top_rpy"   value="${-pi/2} 0 ${pi}"/>
-  <!-- MID-360 몸통 원점에서 내부 IMU 까지 (Livox 공장값) -->
-  <xacro:property name="imu_xyz"   value="0.011 0.02329 -0.04412"/>
-  <material name="grey"><color rgba="0.4 0.4 0.4 0.6"/></material>
+  <xacro:property name="front_xyz" value="0.30 0.0 0.397"/>
+  <xacro:property name="front_rpy" value="0 0 ${pi/2}"/>
+  <xacro:property name="rear_xyz"  value="-0.98 -0.56 0.35"/>
+  <xacro:property name="rear_rpy"  value="0 0 ${-pi/2}"/>
+  <!-- body(=top 라이다 내부 IMU) 에서 본 base_footprint.
+       계산: inverse( T(base_footprint<-top) * T(top<-IMU) )
+       T(top<-IMU) 는 MID-360 공장값 (0.011, 0.02329, -0.04412), 회전 없음. -->
+  <xacro:property name="bf_from_body_xyz" value="-0.011 1.37671 -0.51588"/>
+  <xacro:property name="bf_from_body_rpy" value="${-pi/2} 0 ${-pi}"/>
+  <material name="grey"><color rgba="0.4 0.4 0.4 0.5"/></material>
   <material name="orange"><color rgba="0.9 0.5 0.1 1.0"/></material>
-  <!-- MID-360 한 대를 붙이는 매크로 -->
   <xacro:macro name="mid360" params="name xyz rpy">
     <link name="${name}">
@@ -46,22 +43,35 @@
       </visual>
     </link>
-    <joint name="livox_frame_to_${name}" type="fixed">
-      <parent link="livox_frame"/>
+    <joint name="base_footprint_to_${name}" type="fixed">
+      <parent link="base_footprint"/>
       <child  link="${name}"/>
       <origin xyz="${xyz}" rpy="${rpy}"/>
     </joint>
   </xacro:macro>
-  <!-- ===== 차체 ===== -->
-  <link name="body">
+  <!-- ===== 루트: FAST-LIO 가 내보내는 IMU 프레임 ===== -->
+  <link name="body"/>
+  <!-- 같은 지점에 대한 별칭. IMU 메시지 시각화용. -->
+  <link name="imu_link"/>
+  <joint name="body_to_imu_link" type="fixed">
+    <parent link="body"/><child link="imu_link"/>
+    <origin xyz="0 0 0" rpy="0 0 0"/>
+  </joint>
+  <!-- ===== 차량 기준점 (지면) ===== -->
+  <link name="base_footprint">
     <visual>
       <geometry><box size="${body_length} ${body_width} ${body_height}"/></geometry>
-      <origin xyz="0 0 ${body_height/2 - 0.18}"/>
+      <origin xyz="0 0 ${body_height/2}"/>
       <material name="grey"/>
     </visual>
   </link>
+  <joint name="body_to_base_footprint" type="fixed">
+    <parent link="body"/><child link="base_footprint"/>
+    <origin xyz="${bf_from_body_xyz}" rpy="${bf_from_body_rpy}"/>
+  </joint>
+  <!-- 드라이버가 원시 클라우드 header 에 찍는 이름. 병합 전이라 기하학적
+       의미는 없고, RViz 가 프레임을 못 찾는 것만 막아준다. -->
   <link name="livox_frame"/>
-  <joint name="body_to_livox_frame" type="fixed">
-    <parent link="body"/>
-    <child  link="livox_frame"/>
+  <joint name="base_footprint_to_livox_frame" type="fixed">
+    <parent link="base_footprint"/><child link="livox_frame"/>
     <origin xyz="0 0 0" rpy="0 0 0"/>
   </joint>
@@ -70,10 +80,3 @@
   <xacro:mid360 name="livox_front" xyz="${front_xyz}" rpy="${front_rpy}"/>
   <xacro:mid360 name="livox_rear"  xyz="${rear_xyz}"  rpy="${rear_rpy}"/>
-  <!-- ===== IMU (상단 라이다 내장) ===== -->
-  <link name="imu_link"/>
-  <joint name="livox_top_to_imu" type="fixed">
-    <parent link="livox_top"/>
-    <child  link="imu_link"/>
-    <origin xyz="${imu_xyz}" rpy="0 0 0"/>
-  </joint>
 </robot>

Commit message: 장착 기준을 예전 static TF 로 되돌리고, 정합 검사 스크립트 추가
rbio 값은 base_footprint 에 대해 원점대칭이 아니었다.
  front (0.30, 0, 0.397)  rear (-0.98, -0.56, 0.35)
  합 xy = (-0.68, -0.56)  중점 (-0.34, -0.28)
yaw 는 +90/-90 으로 180도 차이라 방향은 대칭인데 위치 중점이 원점에서
(-0.34, -0.28) 벗어나 있다. rear 와 top 의 y 가 둘 다 정확히 -0.56 이고
차폭 0.952(중심선 +-0.476) 밖으로 8.4cm 나간다. base_footprint 가 차량
중심선이 아닌 것으로 보여 쓰지 않는다.

예전 static TF 값은 대칭이다.
  front (0.697, 0.35, -0.18)  rear (-0.6, -0.34, -0.18)
  합 xy = (0.097, 0.01) ~ 0

top 은 예전 static TF 에 없던 라이다라 rbio 값을 두 기준의 평균 오프셋
(-0.3885, -0.285, 0.5535) 만큼 되돌려 (0.3885, -0.275, 0.8465) 로 추정했다.
front/rear 각각으로 구한 오프셋이 y 에서 13cm 어긋나므로 불확실도가
+-(0.01, 0.065, 0.025) 다. 실측하면 URDF 의 top_xyz 만 고치고 검사
스크립트가 알려주는 대로 extrinsic 을 다시 계산하면 된다.

extrinsic_T: [-0.011, 1.37671, -0.51588] -> [0.3775, 0.82321, -0.23088]

tools/check_frames.py 추가. 같은 기하 정보가 URDF / livox_merge / fast_lio*
세 군데에 있어서 한 곳만 고치면 조용히 어긋난다. 현재 전부 일치.

Co-Authored-By: Claude Opus 5 (1M context) <noreply@anthropic.com>

File: src/description/urdf/vehicle.urdf.xacro (robot description, xacro)
@@ -22,15 +22,27 @@
   <xacro:property name="body_width"  value="0.952"/>
   <xacro:property name="body_height" value="0.60"/>
-  <!-- ===== 라이다 장착 (base_footprint 기준, rbio 값) ===== -->
-  <xacro:property name="top_xyz"   value="0.0 -0.56 1.40"/>
+  <!-- ===== 라이다 장착 (base_footprint 기준) =====
+       front/rear 는 예전 msg_Multi_launch.py 의 static TF 값이다. 이 값들은
+       base_footprint 에 대해 원점대칭이다(합이 xy 로 (0.097, 0.01) ~ 0).
+         front + rear = (0.097, 0.01)   yaw 는 +90 / -90 으로 180도 차이
+       rbio 값은 중점이 (-0.34, -0.28) 로 치우쳐 있고 rear/top 의 y=-0.56 이
+       차폭(0.952) 밖으로 나가서 쓰지 않는다. -->
+  <xacro:property name="front_xyz" value="0.697 0.35 -0.18"/>
+  <xacro:property name="front_rpy" value="0 0 ${pi/2}"/>
+  <xacro:property name="rear_xyz"  value="-0.6 -0.34 -0.18"/>
+  <xacro:property name="rear_rpy"  value="0 0 ${-pi/2}"/>
+  <!-- top: 예전 static TF 에는 이 라이다가 없었다. rbio 값 (0, -0.56, 1.40) 을
+       두 기준의 평균 오프셋 (-0.3885, -0.285, 0.5535) 만큼 되돌린 추정치다.
+       front/rear 각각으로 구한 오프셋이 y 에서 13cm 어긋나므로 이 값의
+       불확실도는 대략 +-(0.01, 0.065, 0.025) 다. 실측하면 여기만 고치면 된다.
+       회전은 실측으로 확인된 값(roll -90, yaw 180). -->
+  <xacro:property name="top_xyz"   value="0.3885 -0.275 0.8465"/>
   <xacro:property name="top_rpy"   value="${-pi/2} 0 ${pi}"/>
-  <xacro:property name="front_xyz" value="0.30 0.0 0.397"/>
-  <xacro:property name="front_rpy" value="0 0 ${pi/2}"/>
-  <xacro:property name="rear_xyz"  value="-0.98 -0.56 0.35"/>
-  <xacro:property name="rear_rpy"  value="0 0 ${-pi/2}"/>
   <!-- body(=top 라이다 내부 IMU) 에서 본 base_footprint.
        계산: inverse( T(base_footprint<-top) * T(top<-IMU) )
-       T(top<-IMU) 는 MID-360 공장값 (0.011, 0.02329, -0.04412), 회전 없음. -->
-  <xacro:property name="bf_from_body_xyz" value="-0.011 1.37671 -0.51588"/>
+       T(top<-IMU) 는 MID-360 공장값 (0.011, 0.02329, -0.04412), 회전 없음.
+       top_xyz 를 고치면 이 값과 fast_lio*/config/mid360.yaml 의 extrinsic_T 를
+       같이 다시 계산해야 한다. -->
+  <xacro:property name="bf_from_body_xyz" value="0.3775 0.82321 -0.23088"/>
   <xacro:property name="bf_from_body_rpy" value="${-pi/2} 0 ${-pi}"/>
   <material name="grey"><color rgba="0.4 0.4 0.4 0.5"/></material>

Commit message: body(=IMU)를 base_footprint 와 같은 x 에 오도록 top_x 확정
body 와 imu_link 의 x 가 base_footprint 와 같아야 한다는 제약을 반영했다.

  R_mount * (0.011, 0.02329, -0.04412) = (-0.011, 0.04412, -0.02329)
  body_x = top_x - 0.011 = 0   ->   top_x = 0.011

  top_xyz      0.3885 -> 0.011
  extrinsic_T  [0.3775, 0.82321, -0.23088] -> [0.0, 0.82321, -0.23088]

검증: base_footprint 기준 body / imu_link 둘 다 x = 0.000 확인.

이 제약이 알려주는 것: rbio 의 top_x 는 0.0 이었고 그게 사실상 정답이었다.
내가 front/rear 평균 오프셋으로 x 를 -0.3885 만큼 보정한 게 틀렸다는 뜻이다.
그런데 front/rear 의 x 는 두 기준 사이에서 실제로 -0.39 차이가 난다. x 에
대해서만 오프셋이 있다가 없다가 하는 셈이라, rbio 값이 이 차량이 아니라
TransferRobot 이라는 다른 플랫폼 기준일 가능성이 높다.

그러면 rbio 에서 신뢰할 수 있는 건 회전(roll -90, yaw 180)뿐이고, 그건 이미
사용자 확인을 받았다. top 의 y, z 는 여전히 추정치로 남는다.

Co-Authored-By: Claude Opus 5 (1M context) <noreply@anthropic.com>

File: src/description/urdf/vehicle.urdf.xacro (robot description, xacro)
@@ -32,10 +32,13 @@
   <xacro:property name="rear_xyz"  value="-0.6 -0.34 -0.18"/>
   <xacro:property name="rear_rpy"  value="0 0 ${-pi/2}"/>
-  <!-- top: 예전 static TF 에는 이 라이다가 없었다. rbio 값 (0, -0.56, 1.40) 을
-       두 기준의 평균 오프셋 (-0.3885, -0.285, 0.5535) 만큼 되돌린 추정치다.
-       front/rear 각각으로 구한 오프셋이 y 에서 13cm 어긋나므로 이 값의
-       불확실도는 대략 +-(0.01, 0.065, 0.025) 다. 실측하면 여기만 고치면 된다.
-       회전은 실측으로 확인된 값(roll -90, yaw 180). -->
-  <xacro:property name="top_xyz"   value="0.3885 -0.275 0.8465"/>
+  <!-- top: 예전 static TF 에는 이 라이다가 없다.
+       x 는 제약으로 확정: body(=내부 IMU)가 base_footprint 와 x 가 같아야 한다.
+       R_mount * (0.011, 0.02329, -0.04412) = (-0.011, 0.04412, -0.02329) 이므로
+       body_x = top_x - 0.011 = 0  ->  top_x = 0.011.
+       y, z 는 아직 추정치다. rbio 값 (0, -0.56, 1.40) 을 front/rear 두 기준의
+       평균 오프셋만큼 되돌린 값이고, front/rear 각각으로 구한 오프셋이 y 에서
+       13cm 어긋나 불확실도가 +-(0.065, 0.025) 다.
+       회전은 실측 확인됨(roll -90, yaw 180). -->
+  <xacro:property name="top_xyz"   value="0.011 -0.275 0.8465"/>
   <xacro:property name="top_rpy"   value="${-pi/2} 0 ${pi}"/>
   <!-- body(=top 라이다 내부 IMU) 에서 본 base_footprint.
@@ -44,5 +47,5 @@
        top_xyz 를 고치면 이 값과 fast_lio*/config/mid360.yaml 의 extrinsic_T 를
        같이 다시 계산해야 한다. -->
-  <xacro:property name="bf_from_body_xyz" value="0.3775 0.82321 -0.23088"/>
+  <xacro:property name="bf_from_body_xyz" value="0.0 0.82321 -0.23088"/>
   <xacro:property name="bf_from_body_rpy" value="${-pi/2} 0 ${-pi}"/>
   <material name="grey"><color rgba="0.4 0.4 0.4 0.5"/></material>

Commit message: body 를 base_footprint 와 같은 중심좌표(x, y)에 오도록 top_y 확정
top 이 누워 있어(roll -90, yaw 180) 내부 IMU 오프셋도 같이 회전한다.
  R_mount * (0.011, 0.02329, -0.04412) = (-0.011, 0.04412, -0.02329)
  body_xy = top_xy + (-0.011, 0.04412) = (0, 0)  ->  top_xy = (0.011, -0.04412)

  top_xyz      0.011 -0.275 0.8465  ->  0.011 -0.04412 0.8465
  extrinsic_T  [0.0, 0.82321, -0.23088]  ->  [0.0, 0.82321, 0.0]

검증(base_footprint 기준):
  body / imu_link  [0.000, 0.000, 0.823]
  livox_top        [0.011, -0.044, 0.847]
  livox_front      [0.697,  0.350, -0.180]
  livox_rear       [-0.600, -0.340, -0.180]

z 는 0 으로 두지 않았다. IMU 는 실제로 마스트 위에 있고, 0 으로 두면 차량
중심에 있다고 모델링되어 회전 시 lever arm 이 사라진다. FAST-LIO 는 IMU
프레임의 자세를 추정하므로 이 값이 틀리면 각속도가 만드는 선가속도를 잘못
보상해서 자세 추정이 틀어진다. 평면화는 tf_2d 가 하므로 nav2 쪽에는 z 가
영향을 주지 않는다.

Co-Authored-By: Claude Opus 5 (1M context) <noreply@anthropic.com>

File: src/description/urdf/vehicle.urdf.xacro (robot description, xacro)
@@ -33,12 +33,14 @@
   <xacro:property name="rear_rpy"  value="0 0 ${-pi/2}"/>
   <!-- top: 예전 static TF 에는 이 라이다가 없다.
-       x 는 제약으로 확정: body(=내부 IMU)가 base_footprint 와 x 가 같아야 한다.
-       R_mount * (0.011, 0.02329, -0.04412) = (-0.011, 0.04412, -0.02329) 이므로
-       body_x = top_x - 0.011 = 0  ->  top_x = 0.011.
-       y, z 는 아직 추정치다. rbio 값 (0, -0.56, 1.40) 을 front/rear 두 기준의
-       평균 오프셋만큼 되돌린 값이고, front/rear 각각으로 구한 오프셋이 y 에서
-       13cm 어긋나 불확실도가 +-(0.065, 0.025) 다.
+       x, y 는 제약으로 확정: body(=top 내부 IMU)가 base_footprint 와 중심좌표
+       (x, y)가 같아야 한다. top 이 누워 있어 내부 IMU 오프셋도 같이 돈다.
+         R_mount * (0.011, 0.02329, -0.04412) = (-0.011, 0.04412, -0.02329)
+         body_xy = top_xy + (-0.011, 0.04412) = (0, 0)
+         -> top_xy = (0.011, -0.04412)
+       z 만 추정치다(0.8465, 오차 +-0.025). z 는 마스트 높이라 x/y 처럼 0 으로
+       둘 수 없다 - 0 으로 두면 IMU 가 차량 중심에 있다고 모델링되어 회전 시
+       lever arm 이 사라지고 FAST-LIO 의 자세 추정이 틀어진다.
        회전은 실측 확인됨(roll -90, yaw 180). -->
-  <xacro:property name="top_xyz"   value="0.011 -0.275 0.8465"/>
+  <xacro:property name="top_xyz"   value="0.011 -0.04412 0.8465"/>
   <xacro:property name="top_rpy"   value="${-pi/2} 0 ${pi}"/>
   <!-- body(=top 라이다 내부 IMU) 에서 본 base_footprint.
@@ -47,5 +49,5 @@
        top_xyz 를 고치면 이 값과 fast_lio*/config/mid360.yaml 의 extrinsic_T 를
        같이 다시 계산해야 한다. -->
-  <xacro:property name="bf_from_body_xyz" value="0.0 0.82321 -0.23088"/>
+  <xacro:property name="bf_from_body_xyz" value="0.0 0.82321 0.0"/>
   <xacro:property name="bf_from_body_rpy" value="${-pi/2} 0 ${-pi}"/>
   <material name="grey"><color rgba="0.4 0.4 0.4 0.5"/></material>
