Commit message: TF 트리를 map->odom->base_link->base_footprint 로 정리
camera_init 과 body 가 사용자 눈에 계속 걸리던 문제. 둘 다 FAST-LIO 가 직접
발행하는 프레임이라 없앨 수는 없지만, 내부 배관으로 밀어내고 실제로 쓰는 체인을
표준 형태로 만들었다.

before
  map ─┬─ camera_init ── body ─┬─ imu_link
       │                       └─ base_footprint ── livox_*
       └─ odom ── base_link            <- 아래에 아무것도 없음

after
  map ─┬─ odom ── base_link ── base_footprint ─┬─ livox_frame
       │                                       ├─ livox_top ── imu_link
       │                                       ├─ livox_front
       │                                       └─ livox_rear
       └─ camera_init ── body ── fastlio_ref   <- 내부 배관, 프레임 하나뿐

차량 모델과 센서가 3D 체인이 아니라 평면화된 2D 체인 아래로 옮겨갔다. nav2 가
쓰는 경로에 시변 3D 변환이 끼지 않아 코스트맵 입장에서도 이쪽이 맞다.

urdf 를 셋으로 쪼갰다.
  mount.xacro            장착값 원본 (아래 둘이 include)
  vehicle.urdf.xacro     base_link 루트. RViz RobotModel 이 보는 쪽
  fastlio_ref.urdf.xacro body 루트. tf_2d.py 가 평면화할 프레임 하나

robot_state_publisher 를 둘 띄운다. TF 는 프레임당 부모가 하나뿐이라 한 URDF 로
두 트리를 못 만든다. 두 번째는 robot_description 을 fastlio_ref_description 으로
remap 해서 RViz 의 RobotModel 과 겹치지 않게 했다.

tf_2d.py 의 평면화 대상: base_footprint -> fastlio_ref.
  tf_2d_bridge started: map->camera_init->fastlio_ref ==> map->odom->base_link

Co-Authored-By: Claude Opus 5 (1M context) <noreply@anthropic.com>

File: src/description/urdf/vehicle.urdf.xacro (robot description, xacro)
@@ -1,52 +1,16 @@
 <?xml version="1.0"?>
 <!--
-  차량 + 센서 장착 형상. TF 의 유일한 출처.
-  장착값 출처: rbio TransferRobot LidarMountCalibration.cpp defaultMountTransform()
-  회전 합성이 yaw*pitch*roll (= Rz*Ry*Rx) 라 URDF rpy 와 같은 관례다.
-  트리가 base_footprint 가 아니라 body 에서 시작하는 이유:
-    FAST-LIO 의 "body" 는 차량 기준점이 아니라 IMU 프레임이다.
-    (publish_frame_body 가 RGBpointBodyLidarToIMU 로 변환해서 body 로 stamp)
-    FAST-LIO 가 camera_init->body 를 이미 내보내므로 body 가 이 URDF 의 루트가
-    되어야 하고, 차량 기준점은 그 아래에 매달린다. TF 는 프레임당 부모가
-    하나뿐이라 반대로는 못 짠다.
-    map ─┬─ camera_init ── body(=IMU, livox_top 내부)
-         │                  └─ base_footprint ─┬─ livox_frame
-         │                                     ├─ livox_top
-         │                                     ├─ livox_front
-         │                                     └─ livox_rear
-         └─ odom ── base_link      <- tf_2d.py 가 base_footprint 를 평면화한 것
+  차량과 센서 형상. 내비게이션이 쓰는 2D 체인 아래에 붙는다.
+    map ── odom ── base_link ── base_footprint ─┬─ livox_frame
+                                                ├─ livox_top ── imu_link
+                                                ├─ livox_front
+                                                └─ livox_rear
+  map->odom, odom->base_link 은 tf_2d.py 가 낸다. base_link 는 이 URDF 의
+  루트이므로 여기서는 발행하지 않는다(부모가 둘이 되면 TF 가 깨진다).
+  FAST-LIO 의 camera_init / body 는 여기 없다. 그쪽은 측위 엔진 내부 프레임이라
+  fastlio_ref.urdf.xacro 로 분리했다.
 -->
 <robot xmlns:xacro="http://www.ros.org/wiki/xacro" name="vehicle">
-  <!-- ===== 차체 치수 (nav2 footprint 와 같은 실측값) ===== -->
-  <xacro:property name="body_length" value="1.62"/>
-  <xacro:property name="body_width"  value="0.952"/>
-  <xacro:property name="body_height" value="0.60"/>
-  <!-- ===== 라이다 장착 (base_footprint 기준) =====
-       front/rear 는 예전 msg_Multi_launch.py 의 static TF 값이다. 이 값들은
-       base_footprint 에 대해 원점대칭이다(합이 xy 로 (0.097, 0.01) ~ 0).
-         front + rear = (0.097, 0.01)   yaw 는 +90 / -90 으로 180도 차이
-       rbio 값은 중점이 (-0.34, -0.28) 로 치우쳐 있고 rear/top 의 y=-0.56 이
-       차폭(0.952) 밖으로 나가서 쓰지 않는다. -->
-  <xacro:property name="front_xyz" value="0.697 0.35 -0.18"/>
-  <xacro:property name="front_rpy" value="0 0 ${pi/2}"/>
-  <xacro:property name="rear_xyz"  value="-0.6 -0.34 -0.18"/>
-  <xacro:property name="rear_rpy"  value="0 0 ${-pi/2}"/>
-  <!-- top: 예전 static TF 에는 이 라이다가 없다.
-       x 는 제약으로 확정: body(=내부 IMU)가 base_footprint 와 x 가 같아야 한다.
-       R_mount * (0.011, 0.02329, -0.04412) = (-0.011, 0.04412, -0.02329) 이므로
-       body_x = top_x - 0.011 = 0  ->  top_x = 0.011.
-       y, z 는 아직 추정치다. rbio 값 (0, -0.56, 1.40) 을 front/rear 두 기준의
-       평균 오프셋만큼 되돌린 값이고, front/rear 각각으로 구한 오프셋이 y 에서
-       13cm 어긋나 불확실도가 +-(0.065, 0.025) 다.
-       회전은 실측 확인됨(roll -90, yaw 180). -->
-  <xacro:property name="top_xyz"   value="0.011 -0.275 0.8465"/>
-  <xacro:property name="top_rpy"   value="${-pi/2} 0 ${pi}"/>
-  <!-- body(=top 라이다 내부 IMU) 에서 본 base_footprint.
-       계산: inverse( T(base_footprint<-top) * T(top<-IMU) )
-       T(top<-IMU) 는 MID-360 공장값 (0.011, 0.02329, -0.04412), 회전 없음.
-       top_xyz 를 고치면 이 값과 fast_lio*/config/mid360.yaml 의 extrinsic_T 를
-       같이 다시 계산해야 한다. -->
-  <xacro:property name="bf_from_body_xyz" value="0.0 0.82321 -0.23088"/>
-  <xacro:property name="bf_from_body_rpy" value="${-pi/2} 0 ${-pi}"/>
+  <xacro:include filename="mount.xacro"/>
   <material name="grey"><color rgba="0.4 0.4 0.4 0.5"/></material>
   <material name="orange"><color rgba="0.9 0.5 0.1 1.0"/></material>
@@ -64,13 +28,8 @@
     </joint>
   </xacro:macro>
-  <!-- ===== 루트: FAST-LIO 가 내보내는 IMU 프레임 ===== -->
-  <link name="body"/>
-  <!-- 같은 지점에 대한 별칭. IMU 메시지 시각화용. -->
-  <link name="imu_link"/>
-  <joint name="body_to_imu_link" type="fixed">
-    <parent link="body"/><child link="imu_link"/>
-    <origin xyz="0 0 0" rpy="0 0 0"/>
-  </joint>
-  <!-- ===== 차량 기준점 (지면) ===== -->
+  <!-- tf_2d.py 가 내보내는 평면화된 차량 프레임 -->
+  <link name="base_link"/>
+  <!-- 차량 기준점. tf_2d 가 이미 z 를 0 으로 눌러 놓으므로 base_link 와 같은
+       지점이다. 모델과 센서를 매다는 자리. -->
   <link name="base_footprint">
     <visual>
@@ -80,7 +39,7 @@
     </visual>
   </link>
-  <joint name="body_to_base_footprint" type="fixed">
-    <parent link="body"/><child link="base_footprint"/>
-    <origin xyz="${bf_from_body_xyz}" rpy="${bf_from_body_rpy}"/>
+  <joint name="base_link_to_base_footprint" type="fixed">
+    <parent link="base_link"/><child link="base_footprint"/>
+    <origin xyz="0 0 0" rpy="0 0 0"/>
   </joint>
   <!-- 드라이버가 원시 클라우드 header 에 찍는 이름. 병합 전이라 기하학적
@@ -91,7 +50,13 @@
     <origin xyz="0 0 0" rpy="0 0 0"/>
   </joint>
-  <!-- ===== 라이다 3대 ===== -->
   <xacro:mid360 name="livox_top"   xyz="${top_xyz}"   rpy="${top_rpy}"/>
   <xacro:mid360 name="livox_front" xyz="${front_xyz}" rpy="${front_rpy}"/>
   <xacro:mid360 name="livox_rear"  xyz="${rear_xyz}"  rpy="${rear_rpy}"/>
+  <!-- 상단 라이다 내장 IMU. FAST-LIO 의 body 프레임이 가리키는 물리적 지점과
+       같은 곳이지만, 이쪽은 URDF 가 모델링한 위치다. -->
+  <link name="imu_link"/>
+  <joint name="livox_top_to_imu" type="fixed">
+    <parent link="livox_top"/><child link="imu_link"/>
+    <origin xyz="${imu_xyz}" rpy="0 0 0"/>
+  </joint>
 </robot>
