Commit message: fast_lio / pcd2pgm 제거에 맞춰 정리, CMP0074 경고 해소
[삭제된 패키지 뒤처리]
매핑용 fast_lio 와 3D->2D 변환 pcd2pgm 이 없어졌다. 주행에는 안 쓰이지만
참조가 남아 있어 정리했다.
  tools/check_frames.py   src/fast_lio/config/mid360.yaml 을 읽다가 죽었다
  .gitignore              src/fast_lio/PCD, Log 항목
  README                  구조도, 맵 만들기 절차

맵을 새로 만들려면 두 패키지를 다시 받아 별도 워크스페이스에서 돌리고 결과물만
navigation/map 으로 옮기면 된다는 안내로 대체했다.

[check_frames.py]
tf_2d.py 가 TF 조회 대신 /Odometry + /map_to_odom 을 받고 ref_from_body_* 를
파라미터로 쓰는 방식으로 바뀌면서 fastlio_ref.urdf.xacro 가 없어졌다. 검사도
URDF 대신 mid360.yaml 의 ref_from_body_* 를 보도록 이미 바뀌어 있었고, 여기서는
삭제된 fast_lio 참조만 걷어냈다. 지금 전부 일치한다.

[CMP0074]
livox_merge / fast_lio_localization 빌드 때마다
"CMake variable PCL_ROOT is set to /usr, For compatibility CMake is ignoring"
경고가 났다. cmake_minimum_required 가 3.8 이라 정책이 OLD 로 잡힌 것이다.
cmake_policy(SET CMP0074 NEW) 를 명시해 없앴다.

Co-Authored-By: Claude Opus 5 (1M context) <noreply@anthropic.com>

File: src/navigation/urdf/mount.xacro (robot description, xacro)
@@ -1,5 +1,5 @@
 <?xml version="1.0"?>
 <!--
-  장착값 한 곳. vehicle.urdf.xacro 와 fastlio_ref.urdf.xacro 가 같이 읽는다.
+  장착값 한 곳. vehicle.urdf.xacro 가 읽는다.
   값을 고치면 반드시 tools/check_frames.py 로 livox_merge / fast_lio 설정과의
   정합을 확인할 것.
@@ -21,7 +21,6 @@
   <!-- MID-360 몸통 원점 -> 내부 IMU (Livox 공장값) -->
   <xacro:property name="imu_xyz"   value="0.011 0.02329 -0.04412"/>
-  <!-- FAST-LIO 의 body(=IMU) 에서 본 차량 기준점.
-       inverse( T(base_footprint<-livox_top) * T(livox_top<-IMU) ) -->
-  <xacro:property name="ref_from_body_xyz" value="0.0 0.82321 -0.23088"/>
-  <xacro:property name="ref_from_body_rpy" value="${-pi/2} 0 ${-pi}"/>
+  <!-- FAST-LIO 의 body(=IMU) 에서 본 차량 기준점은 여기 없다.
+       fast_lio_localization/config/mid360.yaml 의 ref_from_body_* 를 볼 것.
+       (tf_2d.py 가 파라미터로 받는다) -->
 </robot>

File: src/navigation/urdf/vehicle.urdf.xacro (robot description, xacro)
@@ -8,6 +8,7 @@
   map->odom, odom->base_link 은 tf_2d.py 가 낸다. base_link 는 이 URDF 의
   루트이므로 여기서는 발행하지 않는다(부모가 둘이 되면 TF 가 깨진다).
-  FAST-LIO 의 camera_init / body 는 여기 없다. 그쪽은 측위 엔진 내부 프레임이라
-  fastlio_ref.urdf.xacro 로 분리했다.
+  FAST-LIO 의 camera_init / body 는 측위 엔진 내부 프레임이라 TF 에 올리지
+  않는다(debug_tf 로만 켠다). body -> 차량 기준점 extrinsic 은
+  fast_lio_localization/config/mid360.yaml 의 ref_from_body_* 가 든다.
 -->
 <robot xmlns:xacro="http://www.ros.org/wiki/xacro" name="vehicle">

Commit message: URDF 를 지면 기준(REP-120)으로 정리하고 extrinsic 을 일괄 갱신
- base_footprint 를 지면에 두고(base_link 아래 0.5m, bag 의 prior map 바닥면에서 실측)
  세 라이다를 livox_frame(front/rear 중점) 아래로 묶는다
- livox_merge / FAST-LIO extrinsic 은 base_footprint(지면) 기준, tf_2d 의
  ref_from_body 는 base_link 기준으로 분리. check_frames.py 가 URDF 체인을
  합성해 세 설정과 트리 구조 약속을 전부 검사한다
- costmap 용 슬라이스를 지면 위 0.15~2.3m 로, 차체 셀프 반사 크롭 추가
- 주기 ICP 보정(continuous_global_localization) 켬. 꺼두면 초기 정합 이후
  FAST-LIO 드리프트가 영원히 안 잡힌다

Co-Authored-By: Claude Fable 5 <noreply@anthropic.com>

File: src/navigation/urdf/mount.xacro (robot description, xacro)
@@ -6,20 +6,28 @@
 -->
 <robot xmlns:xacro="http://www.ros.org/wiki/xacro">
-  <!-- 차체 치수 (nav2 footprint 와 같은 실측값) -->
+  <!-- 차체 치수 (nav2 footprint 와 같은 실측값).
+       body_height 는 지면에서 차체 윗면까지다. base_footprint 가 지면에 있으므로
+       차체 상자는 base_footprint 위로 그대로 쌓인다. -->
   <xacro:property name="body_length" value="1.62"/>
   <xacro:property name="body_width"  value="0.952"/>
   <xacro:property name="body_height" value="0.60"/>
-  <!-- 라이다 장착 (base_footprint 기준). front/rear 는 원점대칭이다. -->
-  <xacro:property name="front_xyz" value="0.697 0.35 -0.18"/>
+  <!-- base_link(tf_2d 가 z=0 으로 눌러 내는 평면 프레임) 아래 지면까지의 거리.
+       bag 의 prior map 바닥면에서 실측. base_footprint 가 여기에 놓인다. -->
+  <xacro:property name="ground_drop" value="0.50"/>
+  <!-- 라이다 중심 프레임 (base_footprint=지면 기준).
+       front/rear 의 중점이고, z 0.32 는 지면 위 라이다 평면 높이다. -->
+  <xacro:property name="livox_frame_xyz" value="0.0485 0.005 0.32"/>
+  <!-- 라이다 장착 (livox_frame 기준). front/rear 는 정의상 정확히 원점대칭이다. -->
+  <xacro:property name="front_xyz" value="0.6485 0.345 0"/>
   <xacro:property name="front_rpy" value="0 0 ${pi/2}"/>
-  <xacro:property name="rear_xyz"  value="-0.6 -0.34 -0.18"/>
+  <xacro:property name="rear_xyz"  value="-0.6485 -0.345 0"/>
   <xacro:property name="rear_rpy"  value="0 0 ${-pi/2}"/>
-  <!-- top 은 옆으로 눕혀 장착. x, y 는 내부 IMU 가 base_footprint 와 중심좌표를
-       공유하도록 역산한 값이고, z 만 추정치다(오차 +-0.025). -->
-  <xacro:property name="top_xyz"   value="0.011 -0.275 0.8465"/>
+  <!-- top 은 옆으로 눕혀 장착. x 는 내부 IMU 가 base_link 의 x=0 에 오도록
+       역산한 값이고, z 만 추정치다(오차 +-0.025). -->
+  <xacro:property name="top_xyz"   value="-0.0375 -0.28 1.0265"/>
   <xacro:property name="top_rpy"   value="${-pi/2} 0 ${pi}"/>
   <!-- MID-360 몸통 원점 -> 내부 IMU (Livox 공장값) -->
   <xacro:property name="imu_xyz"   value="0.011 0.02329 -0.04412"/>
-  <!-- FAST-LIO 의 body(=IMU) 에서 본 차량 기준점은 여기 없다.
+  <!-- FAST-LIO 의 body(=IMU) 에서 본 base_link 는 여기 없다.
        fast_lio_localization/config/mid360.yaml 의 ref_from_body_* 를 볼 것.
        (tf_2d.py 가 파라미터로 받는다) -->

File: src/navigation/urdf/vehicle.urdf.xacro (robot description, xacro)
@@ -2,12 +2,17 @@
 <!--
   차량과 센서 형상. 내비게이션이 쓰는 2D 체인 아래에 붙는다.
-    map ── odom ── base_link ── base_footprint ─┬─ livox_frame
-                                                ├─ livox_top ── imu_link
-                                                ├─ livox_front
-                                                └─ livox_rear
+    map ── odom ── base_link ── base_footprint ── livox_frame ─┬─ livox_top ── imu_link
+                                (지면)            (라이다 중심) ├─ livox_front
+                                                               └─ livox_rear
   map->odom, odom->base_link 은 tf_2d.py 가 낸다. base_link 는 이 URDF 의
   루트이므로 여기서는 발행하지 않는다(부모가 둘이 되면 TF 가 깨진다).
+  base_link 는 tf_2d.py 의 planarize() 가 z 를 0 으로 눌러 만드는 평면 프레임이라
+  지면이 아니다. 지면은 그보다 ground_drop(0.5m) 아래이고, base_footprint 가
+  REP-120 대로 거기에 놓인다. 따라서 base_footprint 기준 z 는 곧 지면 위 높이다.
+  livox_frame 은 세 라이다를 묶는 중심 프레임으로, front/rear 의 중점이다.
+  (드라이버가 클라우드에 찍는 frame_id 는 livox_top/front/rear 이고
+   livox_frame 은 쓰지 않는다 - multi_MID360_config.json 참조)
   FAST-LIO 의 camera_init / body 는 측위 엔진 내부 프레임이라 TF 에 올리지
-  않는다(debug_tf 로만 켠다). body -> 차량 기준점 extrinsic 은
+  않는다(debug_tf 로만 켠다). body -> base_link extrinsic 은
   fast_lio_localization/config/mid360.yaml 의 ref_from_body_* 가 든다.
 -->
@@ -23,14 +28,13 @@
       </visual>
     </link>
-    <joint name="base_footprint_to_${name}" type="fixed">
-      <parent link="base_footprint"/>
+    <joint name="livox_frame_to_${name}" type="fixed">
+      <parent link="livox_frame"/>
       <child  link="${name}"/>
       <origin xyz="${xyz}" rpy="${rpy}"/>
     </joint>
   </xacro:macro>
-  <!-- tf_2d.py 가 내보내는 평면화된 차량 프레임 -->
+  <!-- tf_2d.py 가 내보내는 평면화된 차량 프레임 (z 는 지면이 아니다) -->
   <link name="base_link"/>
-  <!-- 차량 기준점. tf_2d 가 이미 z 를 0 으로 눌러 놓으므로 base_link 와 같은
-       지점이다. 모델과 센서를 매다는 자리. -->
+  <!-- 지면 투영점. 차체와 센서를 매다는 자리이고, 여기 기준 z = 지면 위 높이. -->
   <link name="base_footprint">
     <visual>
@@ -42,12 +46,11 @@
   <joint name="base_link_to_base_footprint" type="fixed">
     <parent link="base_link"/><child link="base_footprint"/>
-    <origin xyz="0 0 0" rpy="0 0 0"/>
+    <origin xyz="0 0 ${-ground_drop}" rpy="0 0 0"/>
   </joint>
-  <!-- 드라이버가 원시 클라우드 header 에 찍는 이름. 병합 전이라 기하학적
-       의미는 없고, RViz 가 프레임을 못 찾는 것만 막아준다. -->
+  <!-- 세 라이다를 묶는 중심 프레임. front/rear 의 중점이다. -->
   <link name="livox_frame"/>
   <joint name="base_footprint_to_livox_frame" type="fixed">
     <parent link="base_footprint"/><child link="livox_frame"/>
-    <origin xyz="0 0 0" rpy="0 0 0"/>
+    <origin xyz="${livox_frame_xyz}" rpy="0 0 0"/>
   </joint>
   <xacro:mid360 name="livox_top"   xyz="${top_xyz}"   rpy="${top_rpy}"/>

Commit message: 프레임 통합: base_footprint 제거, base_link 를 지면 프레임으로
base_link(평면화 프레임)와 base_footprint(지면)로 기준이 둘로 갈려 있어서
같은 기하가 0.5m 차이 나는 두 벌로 관리됐고, costmap 높이 필터마다 -0.5
보정이 붙었다. base_link 하나를 지면 프레임으로 쓰도록 합친다.

- URDF: base_footprint link/joint 삭제, 차체 상자와 livox_frame 을 base_link 에
  직접 매단다. mount.xacro 의 ground_drop 제거. 라이다 extrinsic 수치는 원래
  지면 기준이라 변경 없음.
- mid360.yaml: ref_from_body_xyz 를 base_link(=지면) 기준으로 재계산
  [0, 0.82321, -0.23088] -> [0, 1.32321, -0.23088]. 이제 extrinsic_T 와 같은
  값이고, check_frames.py 가 둘이 일치하는지도 검사한다.
- livox_merge: output.frame_id = base_link (두 설정 모두).
- frames_check.rviz: Fixed Frame 을 base_link 로.
- /localization 토픽의 child_frame_id 는 rbio 앱 호환을 위해 base_footprint
  문자열을 유지한다(TF 프레임이 아니라 메시지 라벨). tf_2d 의 footprint_frame
  파라미터로 바꿀 수 있다. 앱이 TF 를 직접 조회한다면 identity static TF 필요.

알려진 잔여 사항: 사전지도 PCD 의 바닥면은 map z ≈ -0.385 인데 planarize()
가 z=0 을 강제하므로 RViz 에서 3D prior map 을 겹쳐 보면 차량이 그만큼 떠
보인다. x/y/yaw 와 costmap 높이 필터에는 영향이 없고, 지도를 다시 만들 때
지도 z 를 옮겨 정리한다.

검증: tools/check_frames.py 전부 일치, bag 재생으로 TF 트리(base_footprint
없음)·슬라이스 클라우드 frame_id·costmap 갱신 확인.

Co-Authored-By: Claude Opus 5 (1M context) <noreply@anthropic.com>

File: src/navigation/urdf/mount.xacro (robot description, xacro)
@@ -7,13 +7,10 @@
 <robot xmlns:xacro="http://www.ros.org/wiki/xacro">
   <!-- 차체 치수 (nav2 footprint 와 같은 실측값).
-       body_height 는 지면에서 차체 윗면까지다. base_footprint 가 지면에 있으므로
-       차체 상자는 base_footprint 위로 그대로 쌓인다. -->
+       body_height 는 지면에서 차체 윗면까지다. base_link 가 지면에 있으므로
+       차체 상자는 base_link 위로 그대로 쌓인다. -->
   <xacro:property name="body_length" value="1.62"/>
   <xacro:property name="body_width"  value="0.952"/>
   <xacro:property name="body_height" value="0.60"/>
-  <!-- base_link(tf_2d 가 z=0 으로 눌러 내는 평면 프레임) 아래 지면까지의 거리.
-       bag 의 prior map 바닥면에서 실측. base_footprint 가 여기에 놓인다. -->
-  <xacro:property name="ground_drop" value="0.50"/>
-  <!-- 라이다 중심 프레임 (base_footprint=지면 기준).
+  <!-- 라이다 중심 프레임 (base_link=지면 기준).
        front/rear 의 중점이고, z 0.32 는 지면 위 라이다 평면 높이다. -->
   <xacro:property name="livox_frame_xyz" value="0.0485 0.005 0.32"/>
@@ -24,5 +21,5 @@
   <xacro:property name="rear_rpy"  value="0 0 ${-pi/2}"/>
   <!-- top 은 옆으로 눕혀 장착. x 는 내부 IMU 가 base_link 의 x=0 에 오도록
-       역산한 값이고, z 만 추정치다(오차 +-0.025). -->
+       역산한 값이고, z(지면 기준) 만 추정치다(오차 +-0.025). -->
   <xacro:property name="top_xyz"   value="-0.0375 -0.28 1.0265"/>
   <xacro:property name="top_rpy"   value="${-pi/2} 0 ${pi}"/>

File: src/navigation/urdf/vehicle.urdf.xacro (robot description, xacro)
@@ -2,12 +2,17 @@
 <!--
   차량과 센서 형상. 내비게이션이 쓰는 2D 체인 아래에 붙는다.
-    map ── odom ── base_link ── base_footprint ── livox_frame ─┬─ livox_top ── imu_link
-                                (지면)            (라이다 중심) ├─ livox_front
-                                                               └─ livox_rear
+    map ── odom ── base_link ── livox_frame ─┬─ livox_top ── imu_link
+                     (지면)     (라이다 중심)  ├─ livox_front
+                                              └─ livox_rear
   map->odom, odom->base_link 은 tf_2d.py 가 낸다. base_link 는 이 URDF 의
   루트이므로 여기서는 발행하지 않는다(부모가 둘이 되면 TF 가 깨진다).
-  base_link 는 tf_2d.py 의 planarize() 가 z 를 0 으로 눌러 만드는 평면 프레임이라
-  지면이 아니다. 지면은 그보다 ground_drop(0.5m) 아래이고, base_footprint 가
-  REP-120 대로 거기에 놓인다. 따라서 base_footprint 기준 z 는 곧 지면 위 높이다.
+  base_link 는 tf_2d.py 의 planarize() 가 z 를 0 으로 눌러 만드는 평면 프레임이고,
+  동시에 지면 프레임이다. 즉 base_link 기준 z 는 곧 지면 위 높이이고, 라이다
+  extrinsic / 슬라이스 z / costmap 장애물 높이가 전부 이 하나의 원점을 쓴다.
+  (예전에는 base_link 를 지면보다 0.5m 위에 두고 base_footprint 를 따로 뒀는데,
+   기준이 둘로 갈려 파라미터마다 -0.5 보정이 붙었다. 2026-08-27 에 합쳤다.)
+  주의: 사전지도 PCD 의 바닥면은 map z ≈ -0.385 에 있다. planarize() 가 z=0 을
+  강제하므로 RViz 에서 3D prior map 을 겹쳐 보면 차량이 지도 바닥보다 그만큼
+  떠 보인다. 표시상의 차이일 뿐 x/y/yaw 와 costmap 높이 필터에는 영향이 없다.
   livox_frame 은 세 라이다를 묶는 중심 프레임으로, front/rear 의 중점이다.
   (드라이버가 클라우드에 찍는 frame_id 는 livox_top/front/rear 이고
@@ -34,8 +39,7 @@
     </joint>
   </xacro:macro>
-  <!-- tf_2d.py 가 내보내는 평면화된 차량 프레임 (z 는 지면이 아니다) -->
-  <link name="base_link"/>
-  <!-- 지면 투영점. 차체와 센서를 매다는 자리이고, 여기 기준 z = 지면 위 높이. -->
-  <link name="base_footprint">
+  <!-- tf_2d.py 가 내보내는 평면화된 차량 프레임이자 지면 프레임.
+       차체와 센서를 매다는 자리이고, 여기 기준 z = 지면 위 높이다. -->
+  <link name="base_link">
     <visual>
       <geometry><box size="${body_length} ${body_width} ${body_height}"/></geometry>
@@ -44,12 +48,8 @@
     </visual>
   </link>
-  <joint name="base_link_to_base_footprint" type="fixed">
-    <parent link="base_link"/><child link="base_footprint"/>
-    <origin xyz="0 0 ${-ground_drop}" rpy="0 0 0"/>
-  </joint>
   <!-- 세 라이다를 묶는 중심 프레임. front/rear 의 중점이다. -->
   <link name="livox_frame"/>
-  <joint name="base_footprint_to_livox_frame" type="fixed">
-    <parent link="base_footprint"/><child link="livox_frame"/>
+  <joint name="base_link_to_livox_frame" type="fixed">
+    <parent link="base_link"/><child link="livox_frame"/>
     <origin xyz="${livox_frame_xyz}" rpy="0 0 0"/>
   </joint>

Commit message: livox_merge 제거, pointcloud_concatenate_ros2 로 라이다 3대 TF 병합
- livox_merge 패키지 삭제. 병합은 pointcloud_concatenate_ros2
  (upstream https://github.com/lightinfection/pointcloud_concatenate_ros2
  2e7a23a 기준 + 로컬 수정) 가 TF 로 base_link 기준 수행
- 라이다 드라이버 PointCloud2(xfer_format=0) 로 통일, 실장비/bag 경로 단일화
- FAST-LIO preprocess 에 PointCloud2 절대시각 timestamp 처리 추가,
  mid360.yaml / global_localization.py / RViz 설정 갱신
- mount.xacro 장착값 수정, tools 에 check_lidar_z.py, check_lidar_overlap.py 추가
- motor_node zero_set.py 추가, README 갱신

Co-Authored-By: Claude Fable 5 <noreply@anthropic.com>

File: src/navigation/urdf/mount.xacro (robot description, xacro)
@@ -2,6 +2,7 @@
 <!--
   장착값 한 곳. vehicle.urdf.xacro 가 읽는다.
-  값을 고치면 반드시 tools/check_frames.py 로 livox_merge / fast_lio 설정과의
-  정합을 확인할 것.
+  병합 노드는 이 값을 TF 로 그대로 받아 쓴다(사본 없음). 값을 고치면
+  tools/check_frames.py 로 fast_lio 설정과의 정합을,
+  tools/check_lidar_overlap.py 로 실물과의 정합을 확인할 것.
 -->
 <robot xmlns:xacro="http://www.ros.org/wiki/xacro">
@@ -20,12 +21,8 @@
   <xacro:property name="rear_xyz"  value="-0.6485 -0.345 0"/>
   <xacro:property name="rear_rpy"  value="0 0 ${-pi/2}"/>
-  <!-- top 은 옆으로 눕혀 장착. x 는 내부 IMU 가 base_link 의 x=0 에 오도록
-       역산한 값이고, z(지면 기준) 만 추정치다(오차 +-0.025). -->
-  <xacro:property name="top_xyz"   value="-0.0375 -0.28 1.0265"/>
+  <!-- MID-360 장착 (livox_frame 기준). front/rear 는 정의상 정확히 원점대칭이다. -->
+  <xacro:property name="top_xyz"   value="-0.0375 -0.28 0.1073"/>
   <xacro:property name="top_rpy"   value="${-pi/2} 0 ${pi}"/>
   <!-- MID-360 몸통 원점 -> 내부 IMU (Livox 공장값) -->
   <xacro:property name="imu_xyz"   value="0.011 0.02329 -0.04412"/>
-  <!-- FAST-LIO 의 body(=IMU) 에서 본 base_link 는 여기 없다.
-       fast_lio_localization/config/mid360.yaml 의 ref_from_body_* 를 볼 것.
-       (tf_2d.py 가 파라미터로 받는다) -->
 </robot>

Commit message: 리프트 노드 추가, top 라이다 TF 를 주행/도킹 모드로 전환
- lift_node: RS232 리프트 제어보드(rbio 프로토콜). lift/vertical·lift/horizontal
  (Int32 0 정지/1/2), 시간 기반 구동·완료 판정의 lift_node/move 액션
- navigation/top_tf_switcher.py: top 라이다는 리프트에 달려 z 로 움직이는데 보드에
  위치 피드백이 없다. 양 끝 자세를 바닥 평면 실측으로 잡아 두고 /docking(Bool)
  으로 TF 를 전환한다. 값은 mount.xacro 한 곳(top_xyz/top_rpy, top_dock_*)에서 읽고
  1초마다 재발행해 늦게 붙는 리스너도 수렴시킨다
- mount.xacro: front/top 장착값을 바닥 평면 실측으로 갱신
- bringup: lift:=false 로 리프트 없는 PC 에서도 띄울 수 있게

주의: 도킹모드에서는 FAST-LIO extrinsic(주행모드 유도값)이 실물과 0.6m 어긋난다.

Co-Authored-By: Claude Opus 5 (1M context) <noreply@anthropic.com>

File: src/navigation/urdf/mount.xacro (robot description, xacro)
@@ -1,9 +1,3 @@
 <?xml version="1.0"?>
-<!--
-  장착값 한 곳. vehicle.urdf.xacro 가 읽는다.
-  병합 노드는 이 값을 TF 로 그대로 받아 쓴다(사본 없음). 값을 고치면
-  tools/check_frames.py 로 fast_lio 설정과의 정합을,
-  tools/check_lidar_overlap.py 로 실물과의 정합을 확인할 것.
--->
 <robot xmlns:xacro="http://www.ros.org/wiki/xacro">
   <!-- 차체 치수 (nav2 footprint 와 같은 실측값).
@@ -16,12 +10,19 @@
        front/rear 의 중점이고, z 0.32 는 지면 위 라이다 평면 높이다. -->
   <xacro:property name="livox_frame_xyz" value="0.0485 0.005 0.32"/>
-  <!-- 라이다 장착 (livox_frame 기준). front/rear 는 정의상 정확히 원점대칭이다. -->
-  <xacro:property name="front_xyz" value="0.6485 0.345 0"/>
-  <xacro:property name="front_rpy" value="0 0 ${pi/2}"/>
+  <!-- Front라이다 장착 위치 (livox_frame 기준).-->
+  <xacro:property name="front_xyz" value="0.6485 0.345 0.0825"/>
+  <xacro:property name="front_rpy" value="0.005567 -0.010252 ${pi/2}"/>
+  <!-- Rear라이다 장착 위치 (livox_frame 기준).-->
   <xacro:property name="rear_xyz"  value="-0.6485 -0.345 0"/>
   <xacro:property name="rear_rpy"  value="0 0 ${-pi/2}"/>
-  <!-- MID-360 장착 (livox_frame 기준). front/rear 는 정의상 정확히 원점대칭이다. -->
-  <xacro:property name="top_xyz"   value="-0.0375 -0.28 0.1073"/>
-  <xacro:property name="top_rpy"   value="${-pi/2} 0 ${pi}"/>
+  <!-- Top 라이다 장착 (livox_frame z 0.32 기준).
+       주행모드 지면 위 1.3359 m (rel 1.0159), 도킹모드 1.9346 m (rel 1.6146).
+       URDF 조인트에는 주행모드(top_xyz/top_rpy)가 들어가고, /docking 토픽이
+       true 면 top_tf_switcher.py 가 도킹모드(top_dock_*)로 TF 를 바꿔 낸다.
+   -->
+  <xacro:property name="top_xyz"      value="-0.0375 -0.28 1.0159"/>
+  <xacro:property name="top_rpy"      value="-1.589567 0.009866 ${pi}"/>
+  <xacro:property name="top_dock_xyz" value="-0.0375 -0.28 1.6146"/>
+  <xacro:property name="top_dock_rpy" value="-1.586673 0.009306 ${pi}"/>
   <!-- MID-360 몸통 원점 -> 내부 IMU (Livox 공장값) -->
   <xacro:property name="imu_xyz"   value="0.011 0.02329 -0.04412"/>
